File: Schnuppi.brd (EAGLE design)
At the start: 160 x 100 mm, 17 parts, among them IC1 TTGO_DISP

Commit message: Board Konzept 1 FUMM
Parts:
- removed D2: Power LED, SparkFun-LED:LED_5MM
- added P1, P2, P3, P4, P5: Power LED, SparkFun-LED:LED_5MM
- added R10, R7, R8, R9: (no value), rcl:V234/12
- added S6, S7, S8, S9: TL36PO, switch:TL3XPO
- added X1: 22-23-2041, con-molex:22-23-2041
- moved R6 167.9 mm to (21.6, 63.5), turned to 90 degrees
- moved R3 151.6 mm to (15.2, 63.5), turned to 90 degrees
- moved R2 150.4 mm to (34.3, 63.5), turned to 270 degrees
- moved R1 142.1 mm to (52.1, 80.0), turned to 180 degrees
- moved PAD3 116.2 mm to (21.6, 50.8)
- moved PAD2 106.9 mm to (15.2, 50.8)
- moved RGBLED 63.8 mm to (25.4, 80.0)
- moved PAD1 46.6 mm to (74.9, 80.0)
- moved R4 28.0 mm to (41.9, 63.5)
- moved R5 23.6 mm to (27.9, 63.5), turned to 90 degrees
- moved S4 14.0 mm to (71.1, 25.4), turned to 0 degrees
- moved S5 13.7 mm to (81.3, 25.4), turned to 270 degrees
- moved S3 10.5 mm to (71.1, 15.2), turned to 0 degrees
- moved S2 2.84 mm to (71.1, 35.6), turned to 0 degrees
- moved S1 1.27 mm to (61.0, 25.4)
Connections:
- new net N$14: IC1.22, X1.1
- new net N$18: IC1.5V, X1.4
- new net N$19: IC1.37, S6.2
- new net N$20: IC1.39, S8.2
- new net N$21: IC1.32, S7.2
- new net N$22: IC1.38, S9.2
- new net N$23: R10.1, S7.1
- new net N$24: R9.1, S8.1
- new net N$25: R8.1, S9.1
- new net N$26: R7.1, S6.1
- new net N$27: P1.A, R7.2
- new net N$28: P3.A, R8.2
- new net N$29: P4.A, R9.2
- new net N$30: P5.A, R10.2
- new net N$31: X1.3
- new net N$32: IC1.21, X1.2
- net GND: now also S1.1, S1.2, S2.1, S2.2, S3.1, S3.2, S4.1, S4.2, S5.1, S5.2, S6.3, S7.3, S8.3, S9.3
- net N$12: now also P2.A; no longer D2.A
- net N$13: now also P2.K; no longer D2.K
- net VCC: now also P1.K, P3.K, P4.K, P5.K; no longer S1.1, S1.2, S2.1, S2.2, S3.1, S3.2, S4.1, S4.2, S5.1, S5.2
Routing:
- net VCC: track 0.00 -> 305.1 mm
- net N$18: track 0.00 -> 120.0 mm
- net N$32: track 0.00 -> 82.0 mm
- net N$14: track 0.00 -> 78.8 mm
- net N$11: track 0.00 -> 78.2 mm
- net N$10: track 0.00 -> 73.3 mm
- net N$19: track 0.00 -> 71.8 mm
- net GND: track 0.00 -> 67.4 mm
- net N$13: track 0.00 -> 66.6 mm
- net N$22: track 0.00 -> 66.2 mm
- net N$20: track 0.00 -> 59.9 mm
- net N$21: track 0.00 -> 55.0 mm
- net N$3: track 0.00 -> 43.9 mm
- net N$2: track 0.00 -> 33.2 mm
- net N$4: track 0.00 -> 30.2 mm
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- added copper zone on layer 1, net GND
- added copper zone on layer 16, net GND
Other:
- board size 160 x 100 mm -> 114.3 x 75.9 mm
- board text added: "Schnuppi Projekt"
