File: Schnuppi.sch (EAGLE design)
At the start: 17 parts, among them IC1 TTGO_DISP

Commit message: Board Konzept 1 FUMM
Parts:
- added P1, P3, P4, P5: Power LED, SparkFun-LED:LED5MM
- added R10, R7, R8, R9: (no value), rcl:R-EU_V234/12
- added S6, S7, S8, S9: TL36PO, switch:TL36PO
- added X1: 22-23-2041, con-molex:22-23-2041
- renumbered D2 to P2
Connections:
- new net N$14: IC1.22, X1-1.S
- new net N$18: IC1.5V, X1-4.S
- new net N$19: IC1.37, S6.P
- new net N$20: IC1.39, S8.P
- new net N$21: IC1.32, S7.P
- new net N$22: IC1.38, S9.P
- new net N$23: R10.1, S7.O
- new net N$24: R9.1, S8.O
- new net N$25: R8.1, S9.O
- new net N$26: R7.1, S6.O
- new net N$27: P1.A, R7.2
- new net N$28: P3.A, R8.2
- new net N$29: P4.A, R9.2
- new net N$30: P5.A, R10.2
- new net N$31: X1-3.S
- new net N$32: IC1.21, X1-2.S
- net GND: now also S1.1, S1.2, S2.1, S2.2, S3.1, S3.2, S4.1, S4.2, S5.1, S5.2, S6.S, S7.S, S8.S, S9.S
- net VCC: now also P1.C, P3.C, P4.C, P5.C; no longer S1.1, S1.2, S2.1, S2.2, S3.1, S3.2, S4.1, S4.2, S5.1, S5.2
Other:
- moved on the sheet: R4, R5
